File: pic_programmer.kicad_pcb (KiCad board)
At the start: 4 copper layers, 160 x 99.1 mm, 63 parts, among them J1 DB9-FEMAL, P1 CONN_2, P101 CONN_1, P102 CONN_1, P103 CONN_1, P104 CONN_1, P105 CONN_1, P106 CONN_1, P2 SUPP28, P3 SUPP40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

Commit message: layout changes
Parts:
- moved R12 10.2 mm to (145.5, 122.1)
Routing:
- net /DATA-RB7: track 214.2 -> 224.5 mm
