File: pic_programmer.kicad_sch (KiCad schematic)
At the start: 56 parts, among them J1 DB9-FEMAL, P1 CONN_2, P101 CONN_1, P102 CONN_1, P103 CONN_1, P104 CONN_1, P105 CONN_1, P106 CONN_1, Q1 BC237, Q2 BC307, Q3 BC307, U2 74HC125, U3 7805, U4 LT1373

Commit message: some changes
Parts:
- added U7: 4075, symbol 4xxx_IEEE:4075
- C2: PartNumber (none) -> 12345
- R14: value 470 -> 47
Connections:
- net GND: no longer D7.2 (A)
Other:
- moved on the sheet: D1
